File: wackyPot/wackyPot.sch (KiCad schematic (older format))
At the start: 107 parts, among them J1 USB_B_Micro, J2 Conn_01x02, J3 10K NTC Thermistor, J4 Conn_01x06, SW1 SW_Push, SW2 SW_Push, U1 BQ25895RTW, U2 STM32F411CEUx, U4 ATmega328-AU, U5 DS3231M, U6 MT3608, U7 MIC5205-5.0YM5, U8 GL2576-3.3TA5R, Y1 16MHz

Commit message: Added Reference files. Edited the schematic.
Parts:
- removed C29, C31: 0.1uF, symbol Device:C_Small
- removed C33, C35: 22uF, symbol Device:C_Small
- removed D5: Green, symbol Device:LED_Small
- removed D6: SS34, symbol Device:D_Schottky_Small
- removed J4: Conn_01x06, symbol Connector_Generic:Conn_01x06
- removed JP1: Jumper, symbol Device:Jumper
- removed L2: 10uH, symbol Device:L_Small
- removed L4: 2.2 uH, symbol Device:L_Small
- removed R1: R_Small, symbol Device:R_Small
- removed R10, R11: 130, symbol Device:R_Small
- removed R13: R_Variable, symbol Device:R_Variable
- removed R18: 330, symbol Device:R_Small
- removed R19, R20, R23: 1k, symbol Device:R_Small
- removed R21: 10k, symbol Device:R_Small
- removed R22: 5k, symbol Device:R_Small
- removed SW1: SW_Push, symbol Switch:SW_Push
- removed U4: ATmega328-AU, Package_QFP:TQFP-32_7x7mm_P0.8mm, symbol MCU_Microchip_ATmega:ATmega328-AU
- removed U6: MT3608, Package_TO_SOT_SMD:SOT-23-6, symbol Regulator_Switching:MT3608
- removed U8: GL2576-3.3TA5R, Package_TO_SOT_SMD:TO-263-5_TabPin3, symbol Regulator_Switching:GL2576-3.3TA5R
- removed Y1: 16MHz, symbol Device:Crystal_GND2_Small
- added 8MHz?: Crystal, symbol Device:Crystal
- added C? (x7): 100nF, symbol Device:C_Small
- added C? (x2): 4.3pF, symbol Device:C_Small
- added C? (x2): 20pF, symbol Device:C_Small
- added C?: 2.2uF, symbol Device:C_Small
- added Crystal?: 32.768kHz, symbol Device:Crystal
- added FB?: Ferrite_Bead, symbol Device:Ferrite_Bead
- added J?: Conn_01x06, symbol Connector_Generic:Conn_01x06
- added JP?: Jumper, symbol Device:Jumper
- added R?: 30.1k, symbol Device:R_Small
- added R?: 5.23k, symbol Device:R_Small
- added U?: STM32F411RETx, Package_QFP:LQFP-64_10x10mm_P0.5mm, symbol MCU_ST_STM32F4:STM32F411RETx
- FB?: Brand (none) -> BLM21AG102SN1D
Connections:
- net +3V3: now also C?.1, C?.1, C?.1, C?.1, FB?.1, R?.1, U?.13 (VDDA), U?.19 (VDD), U?.32 (VDD), U?.48 (VDD), U?.64 (VDD)
- net AVDD: now also C?.1, C?.2, FB?.2
- net GND: now also S?.A, S?.B, C?.2, C?.2, C?.2, C?.2, C?.2, C?.2, C?.2, C?.2, C?.2, C?.2, JP?.1, R?.2, U?.18 (VSS), U?.31 (VSS), U?.47 (VSS), U?.63 (VSS); no longer U2.23 (VSS), U2.35 (VSS), U2.47 (VSS), U2.49 (VSS)
- net GNDA: now also C?.1, C?.2, JP?.2, U?.12 (VSSA); no longer U2.8 (VSSA)
- net PC13: no longer U2.2 (PC13)
- net RST_STM32: now reaches S?.C, S?.D
- net RST_STM32: now also C?.1, R?.2, U?.7 (NRST)
- new net: C?.1, Crystal?.2, U?.3 (PC14)
- new net: C?.1, U?.30 (VCAP1)
- new net: C?.1, Crystal?.1, U?.4 (PC15)
- new net: 8MHz?.2, C?.1, U?.5 (PH0)
- new net: 8MHz?.1, C?.1, U?.6 (PH1)
- new net: R?.1, U?.60 (BOOT0)
- new net TCK: U?.49 (PA14)
- new net TMS: U?.46 (PA13)
Other:
- note added: "Nucleo-F411RE suggested filtering.\n"
- note added: "Schematic from Nucleo-FR411RE.\nConfirmed by ScarsFun schematic. \nThe value ferrite bead specification is from ScarsFun.\n\n"
- note added: "Schematic from Nucleo-FR411RE.\nScarsFun schematic uses 22pF instead of 20pF. \nThe LSE crystal specification is from the \nNucleo-FR411RE.\n\n\n"
- note removed: "Input and output ceramic capacitors \nof 22μF are recommended for MT3608 \napplications."
- note removed: "Programming Port"
- note removed: "The recommended values of inductor are 4.7 to\n22μH."
- moved on the sheet: 8MHz1, C1, C12, C13, C14, C15, C16, C17, C2, C25, C3, C30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

Commit message: Moved files to specific folders. Downloaded the correct datasheet and reference manual for STM32F411RET6.
Other:
- note added: "Connect SCL to the logic rail through a 10-kΩ resistor\nConnect SDA to the logic rail through a 10-kΩ resistor\n\nNote: SDA and SCL line is pulled in the STM32."
- note removed: "Connect SCL to the logic rail through a 10-kΩ resistor\nConnect SDA to the logic rail through a 10-kΩ resistor\n\nNote: SDA and SCL line is pulled in the ATmega328."
Changed lines of the file:
@@
 	3350 1400 3900 1400
 Text Notes 2700 5050 0    39   ~ 0
-Connect SCL to the logic rail through a 10-kΩ resistor\nConnect SDA to the logic rail through a 10-kΩ resistor\n\nNote: SDA and SCL line is pulled in the ATmega328.
+Connect SCL to the logic rail through a 10-kΩ resistor\nConnect SDA to the logic rail through a 10-kΩ resistor\n\nNote: SDA and SCL line is pulled in the STM32.
 Wire Notes Line
 	4700 3450 4100 3450
